File: PCB/KiCad/hardware_interface.kicad_pcb (KiCad board)
At the start: 6 copper layers, 86 x 86 mm, 252 parts, among them J1 Reset Header, J10 I2C1, J11 I2C1, J12 TIM1, J13 TIM2, J14 I2C2, J15 I2C2, J16 I2C2, J17 I2C2, J18 3.3V Out, J19 5V Out, J2 SWD Flash, J20 UART1, J21 UART2, J22 UART3, J23 Servo 1, J24 Servo 2, J25 GPIO, J26 Analog 1, J27 Analog 2, J28 USB1, J29 USB2, J3 XT30, J30 LED1, J31 LED2, J4 CAN1, J5 CAN1, J6 SPI1, J7 SPI1, J8 I2C1, J9 I2C1, SW1 Reset, SW2 User Button, U1 STM32F429ZIT6TR, U10 USBLC6-2SC6, U11 TCAN1057AVDRQ1, U12 USBLC6-2SC6, U2 TPS2117DRLR, U3 MIC2039AYM6-TR, U4 OPA2834IDGKR, U5 OPA2834IDGKR, U6 SN74S1051DR, U7 SN74S1051DR, U8 SN74S1051DR, U9 SN74S1051DR, Y1 IQXO-791 8.00MHz

Commit message: PCB: change revision and dates
Other:
- board text added: "CAuDri e.V. - 11/2025"
- board text added: "LARS Hardware Interface v1.1"
- board text removed: "CAuDri e.V. - 06/2025"
Changed lines of the file:
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@@
 		)
 	)
-	(gr_text "LARS Hardware Interface \nv1.0"
+	(gr_text "LARS Hardware Interface \nv1.1"
 		(at 105.4 96.9 0)
 		(layer "F.SilkS")
@@
 		)
 	)
-	(gr_text "CAuDri e.V. - 06/2025"
+	(gr_text "CAuDri e.V. - 11/2025"
 		(at 122.6 89.65 0)
 		(layer "B.SilkS")
@@
 		)
 	)
-	(gr_text "LARS Hardware Interface v1.0\n"
+	(gr_text "LARS Hardware Interface v1.1\n"
 		(at 109 87.05 0)
 		(layer "B.SilkS")
@@
 	)
 	(segment
-		(start 150.8775 100.4)
-		(end 152.1 100.4)
+		(start 152.1 100.4)
+		(end 152.45 100.05)
 		(width 0.2)
 		(layer "F.Cu")
@@
 	)
 	(segment
-		(start 152.1 100.4)
-		(end 152.45 100.05)
+		(start 150.8775 100.4)
+		(end 152.1 100.4)
 		(width 0.2)
 		(layer "F.Cu")
