Commit message: add Lichtblick dummy steering visualization

File: .devcontainer/tools/ros_packages/lars_description/urdf/lars_dummy.urdf (robot description, URDF)
Before this commit: robot lars_dummy, 11 links, 10 joints
Links:
- removed link chassis_link
- removed link front_bumper_link
- removed link front_left_servo_link
- removed link front_right_servo_link
- removed link imu_link
- removed link tof_preview_link
- link base_link: geometry collision box size=0.55 0.32 0.10; visual box size=0.55 0.32 0.10
- link front_left_wheel_link: geometry visual cylinder length=0.045 radius=0.065; visual cylinder length=0.048 radius=0.04
- link front_right_wheel_link: geometry visual cylinder length=0.045 radius=0.065; visual cylinder length=0.048 radius=0.04
- link rear_left_wheel_link: geometry visual cylinder length=0.045 radius=0.065; visual cylinder length=0.048 radius=0.04
- link rear_right_wheel_link: geometry visual cylinder length=0.045 radius=0.065; visual cylinder length=0.048 radius=0.04
Joints:
- removed joint base_to_chassis
- removed joint front_bumper_joint
- removed joint front_left_servo_joint
- removed joint front_right_servo_joint
- removed joint imu_joint
- removed joint tof_preview_joint
- joint front_left_wheel_joint: axis (none) -> 0 0 1; limit (none) -> lower=-0.65 upper=0.65 effort=2.0 velocity=3.0; origin xyz=0 0.035 0 rpy=0 0 0 -> xyz=0.21 0.215 0.055 rpy=0 0 0; parent front_left_servo_link -> base_link; type fixed -> revolute
- joint front_right_wheel_joint: axis (none) -> 0 0 1; limit (none) -> lower=-0.65 upper=0.65 effort=2.0 velocity=3.0; origin xyz=0 -0.035 0 rpy=0 0 0 -> xyz=0.21 -0.215 0.055 rpy=0 0 0; parent front_right_servo_link -> base_link; type fixed -> revolute

Commit message: add IMU and ToF dashboard visualisation

File: .devcontainer/tools/ros_packages/lars_description/urdf/lars_dummy.urdf (robot description, URDF)
Before this commit: robot lars_dummy, 5 links, 4 joints
Links:
- added link tof_front; visual box size=0.07 0.04 0.018; visual cylinder length=0.004 radius=0.009
Joints:
- added joint tof_front_joint: type fixed, parent base_link, child tof_front, origin xyz=0.285 0 0.12 rpy=-1.57079632679 0 -1.57079632679

Commit message: add LARS dummy URDF description

File: .devcontainer/tools/ros_packages/lars_description/urdf/lars_dummy.urdf (robot description, URDF)
Before this commit: robot lars_dummy, 6 links, 5 joints
Links:
- added link vehicle_visualization_frame
Joints:
- added joint vehicle_visualization_joint: type fixed, parent vehicle_visualization_frame, child base_link, origin xyz=0 0 0 rpy=0 0 0
